File: kicad/r-map_v2/Microduino_BASE_DE/Microduino_Base_DE.kicad_pcb (KiCad board)
At the start: 2 copper layers, 25.5 x 27.9 mm, 4 parts, among them P1 CONN_01X02, P2 CONN_01X04, P3 CONN_1x27

Commit message: new kicad hardware project
Parts:
- GS1: value GS3 -> GS4; footprint Connectors:GS3 -> Libreria_PCB_mia:GS4
- P2: footprint Libreria_PCB_mia:AMPMODUII_4pin_90° -> Libreria_PCB_mia:WHURT_4pin_90°_61900411021
- moved P1 0.43 mm to (146.9, 80.4)
- moved P2 0.15 mm to (150.0, 77.0)
Connections:
- net /REF renamed /AREF
- net /TX1 renamed /TX0
Routing:
- net /D9: track 0.00 -> 15.5 mm, vias 0 -> 1
- net +3V3: track 31.1 -> 32.2 mm
Other:
- board text added: "BASE"
- board text added: "D9"
