File: kicad/r-map_v2/Microduino_DIGITALE_DE/Microduino_Digitale_DE.kicad_pcb (KiCad board)
At the start: 2 copper layers, 25.5 x 27.9 mm, 2 parts, among them P1 CONN_1x27, P2 CONN_01X04

Commit message: new kicad hardware project
Parts:
- P2: footprint Libreria_PCB_mia:AMPMODUII_4pin_90° -> Libreria_PCB_mia:WHURT_4pin_90°_61900411021
- moved P2 0.11 mm to (147.6, 77.1)
Connections:
- net /REF renamed /AREF
- net /TX1 renamed /TX0
Other:
- board text added: "DIGITALE"
