File: kicad/r-map_v2/Microduino_HUB_DE/Microduino_HUB_DE.sch (KiCad schematic (older format))
At the start: 50 parts, among them P1 CONN_01X04, P2 CONN_01X04, P3 CONN_01X04, P4 USB_B, P5 CONN_01X04, P6 CONN_01X04, P7 CONN_01X04, P8 CONN_01X04, U1 PCA9517A, U2 PCA9517A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

Commit message: new kicad hardware project
Parts:
- removed U5: LM1117-3.3, symbol LM1117-3.3
- added D1: SK34SMA, Diodes_SMD:D_SMA_Standard, symbol D_Schottky
- added L1: 2,2uH, Libreria_PCB_mia:Induttanza_SMD_2520_Wurth, symbol L
- added R15: 150k, Resistors_SMD:R_1206, symbol R
- added R16: 33k, Resistors_SMD:R_1206, symbol R
- added U5: TLV62569, TO_SOT_Packages_SMD:SOT-23-5, symbol TLV62569
- C13: footprint Capacitors_Tantalum_SMD:CP_Tantalum_Case-A_EIA-3216-18_Hand -> Capacitors_Tantalum_SMD:CP_Tantalum_Case-A_EIA-3216-18_Reflow
- C14: footprint Capacitors_SMD:CP_Elec_8x10 -> Capacitors_THT:CP_Radial_D6.3mm_P2.50mm
- P1, P2, P3, P5, P6, P7, P8: footprint Libreria_PCB_mia:AMPMODUII_4pin -> Libreria_PCB_mia:WURTH_4pin_straight_61900411121
- P4: symbol USB_B -> USB_B-RESCUE-Microduino_HUB_DE
- R1, R10, R11, R12, R13, R14, R2, R3, R4, R5, R6, R7, R8, R9: value 10k -> 2k2
Connections:
- wire segments 195 -> 203
Other:
- note added: "Alimantazione 3,3V 2A"
- note added: "USB per alimentazione\n da fonte esterna"
- note removed: "Alimantazione\n 3,3V 800mA"
- note removed: "USB per alimentazione\n esterna"
- moved on the sheet: C13, C14, C15
