File: kicad/r-map_v2/Microduino_RTC_DE/Microduino_RTC_DE.sch (KiCad schematic (older format))
At the start: 15 parts, among them P1 CONN_1x27, U1 PCF8563, Y1 32,762 kHz

Commit message: new kicad hardware project
Connections:
- net REF renamed AREF
- net TX1 renamed TX0
Changed lines of the file:
@@
 Sheet 1 1
 Title "Microduino RTC DE"
-Date "10 aprile 2017"
+Date "30 luglio 2017"
 Rev "0.0"
 Comp ""
@@
 NoConn ~ 8150 3400
 Text Label 8700 2850 3    60   ~ 0
-REF
+AREF
 Text Label 8800 2850 3    60   ~ 0
 A0
@@
 RX0
 Text Label 10150 3500 2    60   ~ 0
-TX1
+TX0
 Text Label 10150 3600 2    60   ~ 0
 D2
@@
 P 8600 4200
 F 0 "P1" H 8600 4100 50  0000 C CNN
-F 1 "CONN_1x27" V 9500 4600 50  0000 C CNN
+F 1 "CONN_1x27" V 9500 4600 50  0001 C CNN
 F 2 "Libreria_PCB_mia:Upin_27" H 9600 4600 50  0001 C CNN
 F 3 "" H 9600 4600 50  0000 C CNN
