File: kicad/r-map_v2/Microduino_SUPPORTO_DE/Microduino_Supporto_DE.kicad_pcb (KiCad board)
At the start: 2 copper layers, 44 x 72 mm, 1 part, among them P1 CONN_1x27

Commit message: new kicad hardware project
Connections:
- net /REF renamed /AREF
- net /TX1 renamed /TX0
Other:
- board text added: "3V3"
- board text added: "5V"
- board text added: "A0"
- board text added: "A1"
- board text added: "A2"
- board text added: "A3"
- board text added: "A4-SDA"
- board text added: "A5-SCL"
- board text added: "A6"
- board text added: "A7"
- board text added: "AREF"
- board text added: "D10-SS"
- board text added: "D11-MOSI"
- board text added: "D12-MISO"
- board text added: "D13-SCK"
- board text added: "D2"
- board text added: "D3"
- board text added: "D4"
- board text added: "D5"
- board text added: "D6"
- board text added: "D7"
- board text added: "D8"
- board text added: "D9"
- board text added: "DigitEco s.r.l."
- board text added: "GND"
- board text added: "RESET"
- board text added: "RX0-D0"
- board text added: "TX0-D1"
