File: kicad/r-map_v2/Microduino_SUPPORTO_DE/Microduino_Supporto_DE.sch (KiCad schematic (older format))
At the start: 1 part, among them P1 CONN_1x27

Commit message: new kicad hardware project
Connections:
- net REF renamed AREF
- net TX1 renamed TX0
Changed lines of the file:
@@
 encoding utf-8
 Sheet 1 1
-Title "Microduino Supporto DE"
-Date "10 aprile 2017"
+Title "Microduino SUPPORTO DE"
+Date "02 agosto 2017"
 Rev "0.0"
 Comp ""
@@
 NoConn ~ 4450 3200
 Text Label 5000 2650 3    60   ~ 0
-REF
+AREF
 Text Label 5100 2650 3    60   ~ 0
 A0
@@
 RX0
 Text Label 6450 3300 2    60   ~ 0
-TX1
+TX0
 Text Label 6450 3400 2    60   ~ 0
 D2
