File: kicad/r-map_v2/Microduino_GSM_DE/SIM800C_DE/Microduino_SIM800C_DE.kicad_pcb (KiCad board)
At the start: 2 copper layers, 25.5 x 27.9 mm, 13 parts, among them P1 CONN_1x27, P2 CONN_01X06, U1 SIM800C

Commit message: update kicad project
Connections:
- U1 pad 39: /D6 -> /D5
Routing:
- net /D5: track 0.00 -> 16.6 mm, vias 0 -> 1
- net /D6: track 16.2 -> 0.00 mm, vias 1 -> 0
Changed lines of the file:
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@@
     (links 39)
     (no_connects 2)
-    (area 124.255401 58.089999 165.476 104.160001)
+    (area 138.634399 62.662999 164.311401 90.753001)
     (thickness 1.6)
     (drawings 30)
@@
   )
   (setup
-    (last_trace_width 0.25)
+    (last_trace_width 0.5)
     (user_trace_width 0.4)
     (user_trace_width 0.5)
@@
       (net 47 "Net-(U1-Pad38)"))
     (pad 39 smd oval (at -1.095 -8.795 90) (size 1.5 0.6) (layers F.Cu F.Paste F.Mask)
-      (net 23 /D6))
+      (net 22 /D5))
     (pad 40 smd oval (at -2.195 -8.785 90) (size 1.5 0.6) (layers F.Cu F.Paste F.Mask)
       (net 48 "Net-(U1-Pad40)"))
@@
   (segment (start 144.841 71.765) (end 144.841 71.435) (width 0.5) (layer B.Cu) (net 20))
   (segment (start 144.841 71.435) (end 141.2494 67.8434) (width 0.5) (layer B.Cu) (net 20))
-  (segment (start 151.221 82.355) (end 152.516 83.65) (width 0.5) (layer F.Cu) (net 23))
-  (segment (start 141.2494 83.0834) (end 144.9626 83.0834) (width 0.5) (layer B.Cu) (net 23))
-  (via (at 151.221 82.355) (size 1) (drill 0.5) (layers F.Cu B.Cu) (net 23))
-  (segment (start 145.691 82.355) (end 151.221 82.355) (width 0.5) (layer B.Cu) (net 23))
-  (segment (start 144.9626 83.0834) (end 145.691 82.355) (width 0.5) (layer B.Cu) (net 23))
-  (segment (start 152.516 83.65) (end 152.516 87.74) (width 0.5) (layer F.Cu) (net 23))
-  (segment (start 150.316 87.74) (end 149.216 87.74) (width 0.25) (layer F.Cu) (net 25) (status C00000))
+  (segment (start 141.251 80.545) (end 142.461 80.545) (width 0.5) (layer B.Cu) (net 22) (status 400000))
+  (via (at 151.221 82.355) (size 1) (drill 0.5) (layers F.Cu B.Cu) (net 22))
+  (segment (start 152.516 83.65) (end 152.516 87.74) (width 0.5) (layer F.Cu) (net 22))
+  (segment (start 151.221 82.355) (end 152.516 83.65) (width 0.5) (layer F.Cu) (net 22))
+  (segment (start 144.271 82.355) (end 151.221 82.355) (width 0.5) (layer B.Cu) (net 22))
+  (segment (start 142.461 80.545) (end 144.271 82.355) (width 0.5) (layer B.Cu) (net 22))
+  (segment (start 150.316 87.74) (end 149.216 87.74) (width 0.25) (layer F.Cu) (net 25))
   (segment (start 152.411 83.215) (end 157.351 83.215) (width 0.75) (layer B.Cu) (net 25))
   (segment (start 149.631 85.995) (end 152.411 83.215) (width 0.75) (layer B.Cu) (net 25))
