File: kicad/r-map_v2/Microduino_GSM_DE/SIM_shield_DE/Microduino_SIM_shield_DE.sch (KiCad schematic (older format))
At the start: 15 parts, among them P1 CONN_1x27, P2 CONN_01X06, U1 TLV62569, U2 ESDA6V1-5W6

Commit message: kicad schemas update
Parts:
- removed C1: 100uF, Capacitors_Tantalum_SMD:CP_Tantalum_Case-B_EIA-3528-21_Reflow, symbol CP
- added C1: 4,7uF, Capacitors_SMD:C_0805, symbol C
- added C2, C5: 100nF, Capacitors_SMD:C_0805, symbol C
- added C3, C4: 10uF, Capacitors_SMD:C_0805, symbol C
- added R2: 10k, Resistors_SMD:R_0805, symbol R
- L1: value 2,2 uH -> 1 uH; footprint Libreria_PCB_mia:Induttanza_SMD_2520_Wurth -> Libreria_PCB_mia:Induttanza_SMD_3030_Vishay
- R1: renamed from R2; value 56k -> 100k
- R3: renamed from R1; value 330k -> 560k
- R4: renamed from R3; value 22 -> 56
- R5: renamed from R4; value 22 -> 56
- R6: renamed from R5; value 22 -> 56
- renumbered C2 to C6, C3 to C7, C4 to C8
Connections:
- net +5V: now also C1.1, C2.1
- net GND: now also C1.2, C2.2, C3.2, C4.2, C5.2
- net VBAT: now also C3.1, C4.1, C5.1
- net at R1.1, U1.5 (FB): now also R2.2; no longer R3.2
- net VRTC: no longer names the net of P2.2 (P2)
- new net: R2.1, R3.2
- no-connect marks 26 -> 27
Other:
- note added: "VBAT = 4,02 volt"
- note removed: "VBAT = 4,14 volt"
- moved on the sheet: C6, C7, C8, L1, P1, R1, R3, U1
